File: my_keypad.kicad_sch (KiCad schematic)
At the start: 20 parts, among them SW1 SW_Push, U1 ATmega32U4-A, Y1 Crystal_GND24_Small

Commit message: finish footprints/sch
Parts:
- MX1, MX2: footprint (none) -> MX_Alps_Hybrid:MX-1U-NoLED
- SW1: footprint (none) -> random-keyboard-parts:SKQG-1155865
- USB1: footprint (none) -> random-keyboard-parts:Molex-0548190589
Changed lines of the file:
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@@
       (effects (font (size 0.508 0.508)))
     )
-    (property "Footprint" "" (at 150.495 76.835 0)
+    (property "Footprint" "MX_Alps_Hybrid:MX-1U-NoLED" (at 150.495 76.835 0)
       (effects (font (size 1.524 1.524)) hide)
     )
@@
       (effects (font (size 1.524 1.524)))
     )
-    (property "Footprint" "" (at 153.67 43.18 0)
+    (property "Footprint" "random-keyboard-parts:Molex-0548190589" (at 153.67 43.18 0)
       (effects (font (size 1.524 1.524)) hide)
     )
@@
       (effects (font (size 1.27 1.27)))
     )
-    (property "Footprint" "" (at 62.23 26.67 0)
+    (property "Footprint" "random-keyboard-parts:SKQG-1155865" (at 62.23 26.67 0)
       (effects (font (size 1.27 1.27)) hide)
     )
@@
       (effects (font (size 0.508 0.508)))
     )
-    (property "Footprint" "" (at 161.925 76.835 0)
-      (effects (font (size 1.524 1.524)) hide)
-    )
+    (property "Footprint" "MX_Alps_Hybrid:MX-1U-NoLED" (at 161.925 76.835 0)
+      (effects (font (size 1.524 1.524)) hide)
+    )
