File: _autosave-my_keypad.kicad_pcb (KiCad board)
At the start: 2 copper layers, 78.8 x 36.8 mm, 20 parts, among them SW1 SW_Push, U1 ATmega32U4-A, Y1 Crystal_GND24_Small

Commit message: added ground fill
Routing:
- net COL1: track 0.00 -> 38.8 mm, vias 0 -> 1
- net COL0: track 0.00 -> 32.0 mm, vias 0 -> 1
- net ROW0: track 44.8 -> 49.8 mm
- net Net-(U1-D+): track 22.5 -> 23.7 mm
- added copper zone on B.Cu, net GND
Other:
- outline, holes or cut-outs redrawn
Changed lines of the file:
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@@
   (gr_arc (start 66.04 109.22) (mid 65.141974 108.848026) (end 64.77 107.95)
-    (stroke (width 0.1) (type default)) (layer "Edge.Cuts"))
-  (gr_line (start 105.41 91.44) (end 105.41 109.22)
     (stroke (width 0.1) (type default)) (layer "Edge.Cuts"))
   (segment (start 84.29375 96.04375) (end 84.856806 96.606806) (width 0.254) (layer "B.Cu") (net 1))
@@
   (segment (start 90.296 85.436) (end 90.269 85.463) (width 0.254) (layer "B.Cu") (net 5))
   (segment (start 93.741 85.436) (end 93.641 85.436) (width 0.254) (layer "B.Cu") (net 5))
-  (segment (start 99.03 96.52) (end 105.156 96.52) (width 0.254) (layer "B.Cu") (net 6))
-  (segment (start 122.429 84.327) (end 110.236 96.52) (width 0.254) (layer "B.Cu") (net 6))
-  (segment (start 123.317 84.327) (end 122.429 84.327) (width 0.254) (layer "B.Cu") (net 6))
-  (segment (start 105.156 96.52) (end 105.283 96.52) (width 0.254) (layer "B.Cu") (net 6))
+  (segment (start 110.236 96.52) (end 99.03 96.52) (width 0.254) (layer "B.Cu") (net 6))
   (segment (start 140.969 85.852) (end 142.494 84.327) (width 0.254) (layer "B.Cu") (net 6))
   (segment (start 123.317 84.327) (end 123.951 84.327) (width 0.254) (layer "B.Cu") (net 6))
   (segment (start 125.476 85.852) (end 140.969 85.852) (width 0.254) (layer "B.Cu") (net 6))
+  (segment (start 123.317 84.327) (end 122.429 84.327) (width 0.254) (layer "B.Cu") (net 6))
+  (segment (start 122.429 84.327) (end 110.236 96.52) (width 0.254) (layer "B.Cu") (net 6))
   (segment (start 123.951 84.327) (end 125.476 85.852) (width 0.254) (layer "B.Cu") (net 6))
   (segment (start 119.705 77.415) (end 123.317 81.027) (width 0.254) (layer "B.Cu") (net 7))
@@
   (segment (start 67.31 84.035) (end 71.73 79.615) (width 0.254) (layer "B.Cu") (net 9))
   (segment (start 71.73 79.615) (end 71.73 78.74) (width 0.254) (layer "B.Cu") (net 9))
+  (segment (start 109.728 98.031866) (end 109.728 98.0465) (width 0.254) (layer "F.Cu") (net 10))
+  (segment (start 111.125 79.375) (end 111.125 96.634866) (width 0.254) (layer "F.Cu") (net 10))
+  (segment (start 111.125 96.634866) (end 109.728 98.031866) (width 0.254) (layer "F.Cu") (net 10))
+  (via (at 109.728 98.0465) (size 0.8) (drill 0.4) (layers "F.Cu" "B.Cu") (net 10))
+  (segment (start 109.6545 98.12) (end 99.03 98.12) (width 0.254) (layer "B.Cu") (net 10))
+  (segment (start 112.435 78.065) (end 111.125 79.375) (width 0.254) (layer "B.Cu") (net 10))
+  (segment (start 112.435 77.915) (end 112.435 78.065) (width 0.254) (layer "B.Cu") (net 10))
+  (segment (start 109.728 98.0465) (end 109.6545 98.12) (width 0.254) (layer "B.Cu") (net 10))
+  (segment (start 130.175 79.375) (end 129.413 79.375) (width 0.254) (layer "F.Cu") (net 11))
+  (segment (start 129.413 79.375) (end 111.252 97.536) (width 0.254) (layer "F.Cu") (net 11))
+  (via (at 111.252 97.536) (size 0.8) (drill 0.4) (layers "F.Cu" "B.Cu") (net 11))
+  (segment (start 111.036 97.32) (end 99.03 97.32) (width 0.254) (layer "B.Cu") (net 11))
+  (segment (start 111.252 97.536) (end 111.036 97.32) (width 0.254) (layer "B.Cu") (net 11))
   (segment (start 102.1795 101.32) (end 99.03 101.32) (width 0.254) (layer "B.Cu") (net 12))
   (segment (start 102.728 101.8685) (end 102.1795 101.32) (width 0.254) (layer "B.Cu") (net 12))
@@
   (segment (start 73.33 81.87075) (end 73.63925 81.87075) (width 0.2) (layer "B.Cu") (net 13))
   (segment (start 73.63925 81.87075) (end 74.676 82.9075) (width 0.2) (layer "B.Cu") (net 13))
-  (segment (start 83.34375 99.21875) (end 74.6125 90.4875) (width 0.254) (layer "B.Cu") (net 14))
-  (segment (start 86.51875 99.21875) (end 83.34375 99.21875) (width 0.254) (layer "B.Cu") (net 14))
-  (segment (start 74.6125 90.4875) (end 74.6125 84.796) (width 0.254) (layer "B.Cu") (net 14))
-  (segment (start 87.63 98.92) (end 86.8175 98.92) (width 0.254) (layer "B.Cu") (net 14))
+  (segment (start 82.156 98.92) (end 87.63 98.92) (width 0.254) (layer "B.Cu") (net 14))
+  (segment (start 73.66 87.63) (end 73.66 90.424) (width 0.254) (layer "B.Cu") (net 14))
+  (segment (start 74.676 84.7325) (end 74.676 86.614) (width 0.254) (layer "B.Cu") (net 14))
+  (segment (start 74.676 86.614) (end 73.66 87.63) (width 0.254) (layer "B.Cu") (net 14))
   (segment (start 74.6125 84.796) (end 74.676 84.7325) (width 0.254) (layer "B.Cu") (net 14))
-  (segment (start 86.8175 98.92) (end 86.51875 99.21875) (width 0.254) (layer "B.Cu") (net 14))
+  (segment (start 73.66 90.424) (end 82.156 98.92) (width 0.254) (layer "B.Cu") (net 14))
   (segment (start 72.53 82.25125) (end 72.53 78.74) (width 0.2) (layer "B.Cu") (net 15))
   (segment (start 71.77625 82.25125) (end 71.12 82.9075) (width 0.2) (layer "B.Cu") (net 15))
   (segment (start 72.53 82.25125) (end 71.77625 82.25125) (width 0.2) (layer "B.Cu") (net 15))
-  (segment (start 86.81125 99.72) (end 86.51875 100.0125) (width 0.254) (layer "B.Cu") (net 16))
-  (segment (start 86.51875 100.0125) (end 83.34375 100.0125) (width 0.254) (layer "B.Cu") (net 16))
-  (segment (start 83.34375 100.0125) (end 71.12 87.78875) (width 0.254) (layer "B.Cu") (net 16))
-  (segment (start 71.12 87.78875) (end 71.12 84.7325) (width 0.254) (layer "B.Cu") (net 16))
-  (segment (start 87.63 99.72) (end 86.81125 99.72) (width 0.254) (layer "B.Cu") (net 16))
+  (segment (start 71.12 84.7325) (end 71.12 86.36) (width 0.254) (layer "B.Cu") (net 16))
+  (segment (start 71.12 86.36) (end 72.39 87.63) (width 0.254) (layer "B.Cu") (net 16))
+  (segment (start 72.39 87.63) (end 72.39 90.17) (width 0.254) (layer "B.Cu") (net 16))
+  (segment (start 72.39 90.17) (end 81.94 99.72) (width 0.254) (layer "B.Cu") (net 16))
+  (segment (start 81.94 99.72) (end 87.63 99.72) (width 0.254) (layer "B.Cu") (net 16))
   (segment (start 79.375 97.63125) (end 75.40625 101.6) (width 0.254) (layer "F.Cu") (net 17))
   (segment (start 79.375 89.69375) (end 79.375 97.63125) (width 0.254) (layer "F.Cu") (net 17))
@@
   (segment (start 80.617 89.635) (end 79.43375 89.635) (width 0.254) (layer "B.Cu") (net 17))
   (segment (start 75.40625 101.6) (end 73.64 101.6) (width 0.254) (layer "B.Cu") (net 17))
+  (zone (net 2) (net_name "GND") (layer "B.Cu") (hatch edge 0.5)
+    (connect_pads (clearance 0.5))
+    (min_thickness 0.25) (filled_areas_thickness no)
+    (fill (thermal_gap 0.5) (thermal_bridge_width 0.5) (island_removal_mode 2) (island_area_min 10))
+    (polygon
+      (pts
+        (xy 65.532 73.152)
+        (xy 105.156 73.152)
+        (xy 105.156 109.22)
+        (xy 65.532 109.22)
+      )
+    )
+  )
 )
