File: my_keypad.kicad_pcb (KiCad board)
At the start: 2 copper layers, 78.8 x 36.8 mm, 20 parts, among them SW1 SW_Push, U1 ATmega32U4-A, Y1 Crystal_GND24_Small

Commit message: fixed errors
Parts:
- C1, SW1: moved to B.Cu
- moved C3 7.24 mm to (83.3, 103.1), turned to -90 degrees
- moved C1 1.82 mm to (83.3, 96.0), turned to 180 degrees
- moved R2 1.52 mm to (74.7, 83.8), turned to -90 degrees
- moved R3 1.27 mm to (71.1, 83.8), turned to -90 degrees
- moved C6 0.32 mm to (99.2, 86.5)
- moved USB1 0.16 mm to (73.3, 74.1)
- turned SW1 to 180 degrees
Routing:
- net GND: track 0.00 -> 144.8 mm
- net +5V: track 0.00 -> 107.5 mm, vias 0 -> 5
- net ROW0: track 0.00 -> 49.8 mm
- net COL1: track 0.00 -> 38.8 mm, vias 0 -> 1
- net COL0: track 0.00 -> 32.0 mm, vias 0 -> 1
- net Net-(U1-~{RESET}): track 0.00 -> 27.9 mm, vias 0 -> 2
- net Net-(U1-D-): track 0.00 -> 25.2 mm
- net Net-(U1-D+): track 0.00 -> 23.6 mm
- net VCC: track 0.00 -> 12.0 mm
- net Net-(U1-XTAL2): track 0.00 -> 10.3 mm
- net Net-(U1-XTAL1): track 0.00 -> 9.91 mm
- net Net-(D2-A): track 0.00 -> 7.51 mm
- net Net-(D1-A): track 0.00 -> 7.38 mm
- net D-: track 0.00 -> 5.19 mm
- net D+: track 0.00 -> 4.91 mm
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- added copper zone on B.Cu, net GND
Other:
- outline, holes or cut-outs redrawn
- board text added: "nguyen"
